Commit message: fix: fix file names (#6)
Signed-off-by: Kenji Miyake <kenji.miyake@tier4.jp>

File: sample_vehicle_description/urdf/vehicle.xacro (robot description, xacro)
@@ -11,5 +11,5 @@
       <origin xyz="${vehicle_info['/**']['ros__parameters']['wheel_base']/2.0} 0 0" rpy="${pi/2.0} 0 ${pi}"/>
       <geometry>
-        <mesh filename="package://sample_vehicle_description/mesh/sample_vehicle.dae" scale="1 1 1"/>
+        <mesh filename="package://sample_vehicle_description/mesh/lexus.dae" scale="1 1 1"/>
       </geometry>
     </visual>

Commit message: ci(pre-commit): update pre-commit-hooks-ros (#16)
* ci(pre-commit): update pre-commit-hooks-ros

Signed-off-by: Kenji Miyake <kenji.miyake@tier4.jp>

* ci(pre-commit): autofix

* Update .pre-commit-config.yaml

* Update .pre-commit-config.yaml

Co-authored-by: pre-commit-ci[bot] <66853113+pre-commit-ci[bot]@users.noreply.github.com>

File: sample_vehicle_description/urdf/vehicle.xacro (robot description, xacro)
@@ -2,8 +2,5 @@
 <robot xmlns:xacro="http://ros.org/wiki/xacro">
   <!-- load parameter -->
-  <xacro:property
-    name="vehicle_info"
-    value="${load_yaml('$(find sample_vehicle_description)/config/vehicle_info.param.yaml')}"
-  />
+  <xacro:property name="vehicle_info" value="${load_yaml('$(find sample_vehicle_description)/config/vehicle_info.param.yaml')}"/>
   <!-- vehicle body -->
   <link name="base_link">

Commit message: config vehicle description

File: sample_vehicle_description/urdf/vehicle.xacro (robot description, xacro)
@@ -8,7 +8,20 @@
       <origin xyz="${vehicle_info['/**']['ros__parameters']['wheel_base']/2.0} 0 0" rpy="${pi/2.0} 0 ${pi}"/>
       <geometry>
-        <mesh filename="package://sample_vehicle_description/mesh/lexus.dae" scale="1 1 1"/>
+        <box size="0 0 0"/>
       </geometry>
     </visual>
   </link>
+  <link name="car_link">
+		<visual>
+		    <origin xyz="0 0 0" rpy="0 0 0"/>
+			<geometry>
+				<box size="0.403 0.306 0.262"/>
+			</geometry>
+		</visual>
+	</link>
+  <joint name="car_joint" type="fixed">
+    	<parent link="base_link"/>
+    	<child link="car_link"/>
+    	<origin xyz="1.5825 0 1.3155" rpy="0 0 0"/>
+	</joint>
 </robot>

Commit message: fix vehicle.xacro

File: sample_vehicle_description/urdf/vehicle.xacro (robot description, xacro)
@@ -16,5 +16,5 @@
 		    <origin xyz="0 0 0" rpy="0 0 0"/>
 			<geometry>
-				<box size="0.403 0.306 0.262"/>
+				<box size="0.421 0.306 0.262"/>
 			</geometry>
 		</visual>
@@ -23,5 +23,5 @@
     	<parent link="base_link"/>
     	<child link="car_link"/>
-    	<origin xyz="1.5825 0 1.3155" rpy="0 0 0"/>
+    	<origin xyz="0.1593 0 0.131" rpy="0 0 0"/>
 	</joint>
 </robot>
